File: HMI.sch (KiCad schematic (older format))
At the start: 12 parts, among them SW501 SW_Push, SW502 SW_Push, SW503 SW_Push

Commit message: finish schematics. add componants, find right chip, firest verification OK, ready for routing
Parts:
- LED501, LED502, LED503: footprint (none) -> LEDs:LED_D5.0mm
- R501, R502, R503, R504, R505, R506: footprint (none) -> Resistors_THT:R_Axial_DIN0207_L6.3mm_D2.5mm_P7.62mm_Horizontal
- SW501, SW502, SW503: footprint (none) -> Buttons_Switches_THT:SW_PUSH_6mm
Changed lines of the file:
@@
 F 0 "LED501" H 2250 3100 50  0000 C CNN
 F 1 "LED" H 2350 2950 50  0000 C CNN
-F 2 "" H 2250 3000 50  0001 C CNN
+F 2 "LEDs:LED_D5.0mm" H 2250 3000 50  0001 C CNN
 F 3 "" H 2250 3000 50  0001 C CNN
 	1    2250 3000
@@
 F 0 "LED502" H 2450 3100 50  0000 C CNN
 F 1 "LED" H 2550 2950 50  0000 C CNN
-F 2 "" H 2450 3000 50  0001 C CNN
+F 2 "LEDs:LED_D5.0mm" H 2450 3000 50  0001 C CNN
 F 3 "" H 2450 3000 50  0001 C CNN
 	1    2450 3000
@@
 F 0 "LED503" H 2650 3100 50  0000 C CNN
 F 1 "LED" H 2750 2950 50  0000 C CNN
-F 2 "" H 2650 3000 50  0001 C CNN
+F 2 "LEDs:LED_D5.0mm" H 2650 3000 50  0001 C CNN
 F 3 "" H 2650 3000 50  0001 C CNN
 	1    2650 3000
@@
 F 0 "R504" V 2330 2650 50  0000 C CNN
 F 1 "R" V 2250 2650 50  0000 C CNN
-F 2 "" V 2180 2650 50  0001 C CNN
+F 2 "Resistors_THT:R_Axial_DIN0207_L6.3mm_D2.5mm_P7.62mm_Horizontal" V 2180 2650 50  0001 C CNN
 F 3 "" H 2250 2650 50  0001 C CNN
 	1    2250 2650
@@
 F 0 "R505" V 2530 2650 50  0000 C CNN
 F 1 "R" V 2450 2650 50  0000 C CNN
-F 2 "" V 2380 2650 50  0001 C CNN
+F 2 "Resistors_THT:R_Axial_DIN0207_L6.3mm_D2.5mm_P7.62mm_Horizontal" V 2380 2650 50  0001 C CNN
 F 3 "" H 2450 2650 50  0001 C CNN
 	1    2450 2650
@@
 F 0 "R506" V 2730 2650 50  0000 C CNN
 F 1 "R" V 2650 2650 50  0000 C CNN
-F 2 "" V 2580 2650 50  0001 C CNN
+F 2 "Resistors_THT:R_Axial_DIN0207_L6.3mm_D2.5mm_P7.62mm_Horizontal" V 2580 2650 50  0001 C CNN
 F 3 "" H 2650 2650 50  0001 C CNN
 	1    2650 2650
@@
 $EndComp
 $Comp
-L GND #PWR015
+L GND #PWR019
 U 1 1 5A7A4E6C
 P 2450 3300
-F 0 "#PWR015" H 2450 3050 50  0001 C CNN
+F 0 "#PWR019" H 2450 3050 50  0001 C CNN
 F 1 "GND" H 2450 3150 50  0000 C CNN
 F 2 "" H 2450 3300 50  0001 C CNN
@@
 F 0 "R501" V 3330 2500 50  0000 C CNN
 F 1 "R" V 3250 2500 50  0000 C CNN
-F 2 "" V 3180 2500 50  0001 C CNN
+F 2 "Resistors_THT:R_Axial_DIN0207_L6.3mm_D2.5mm_P7.62mm_Horizontal" V 3180 2500 50  0001 C CNN
 F 3 "" H 3250 2500 50  0001 C CNN
 	1    3250 2500
@@
 F 0 "R502" V 3830 2500 50  0000 C CNN
 F 1 "R" V 3750 2500 50  0000 C CNN
-F 2 "" V 3680 2500 50  0001 C CNN
+F 2 "Resistors_THT:R_Axial_DIN0207_L6.3mm_D2.5mm_P7.62mm_Horizontal" V 3680 2500 50  0001 C CNN
 F 3 "" H 3750 2500 50  0001 C CNN
 	1    3750 2500
@@
 $EndComp
 $Comp
-L GND #PWR016
+L GND #PWR020
 U 1 1 5A7A4E85
 P 3500 3300
-F 0 "#PWR016" H 3500 3050 50  0001 C CNN
+F 0 "#PWR020" H 3500 3050 50  0001 C CNN
 F 1 "GND" H 3500 3150 50  0000 C CNN
 F 2 "" H 3500 3300 50  0001 C CNN
@@
 F 0 "R503" V 4430 2500 50  0000 C CNN
 F 1 "R" V 4350 2500 50  0000 C CNN
-F 2 "" V 4280 2500 50  0001 C CNN
+F 2 "Resistors_THT:R_Axial_DIN0207_L6.3mm_D2.5mm_P7.62mm_Horizontal" V 4280 2500 50  0001 C CNN
 F 3 "" H 4350 2500 50  0001 C CNN
 	1    4350 2500
@@
 	4350 2250 4350 2350
 Connection ~ 3750 2250
-Wire Wire Line
-	4350 2650 4350 2800
-Wire Wire Line
-	4450 2700 4350 2700
-Connection ~ 4350 2700
 Wire Notes Line
 	2100 4950 3700 4950
@@
 F 0 "SW501" H 3300 3100 50  0000 L CNN
 F 1 "SW_Push" H 3250 2940 50  0000 C CNN
-F 2 "" H 3250 3200 50  0001 C CNN
+F 2 "Buttons_Switches_THT:SW_PUSH_6mm" H 3250 3200 50  0001 C CNN
 F 3 "" H 3250 3200 50  0001 C CNN
 	1    3250 3000
@@
 F 0 "SW502" H 3800 3100 50  0000 L CNN
 F 1 "SW_Push" H 3750 2940 50  0000 C CNN
-F 2 "" H 3750 3200 50  0001 C CNN
+F 2 "Buttons_Switches_THT:SW_PUSH_6mm" H 3750 3200 50  0001 C CNN
 F 3 "" H 3750 3200 50  0001 C CNN
 	1    3750 3000
@@
 F 0 "SW503" H 4400 3100 50  0000 L CNN
 F 1 "SW_Push" H 4350 2940 50  0000 C CNN
-F 2 "" H 4350 3200 50  0001 C CNN
+F 2 "Buttons_Switches_THT:SW_PUSH_6mm" H 4350 3200 50  0001 C CNN
 F 3 "" H 4350 3200 50  0001 C CNN
 	1    4350 3000
@@
 Text GLabel 4450 2700 2    60   Input ~ 0
 P_RESET
+Wire Wire Line
+	4350 2650 4350 2800
+Wire Wire Line
+	4450 2700 4350 2700
+Connection ~ 4350 2700
 $EndSCHEMATC
