File: IO.sch (KiCad schematic (older format))
At the start: 21 parts, among them J201 Conn_01x06, J202 Conn_01x06

Commit message: finish schematics. add componants, find right chip, firest verification OK, ready for routing
Parts:
- added J203: Conn_01x06, Pin_Headers:Pin_Header_Straight_1x06_Pitch2.54mm, symbol Conn_01x06
- added J204: Conn_01x02, Pin_Headers:Pin_Header_Straight_1x02_Pitch2.54mm, symbol Conn_01x02
- added J205: Conn_01x04, Socket_Strips:Socket_Strip_Straight_1x04_Pitch2.54mm, symbol Conn_01x04
- R_pullup_reset_esp_1: footprint (none) -> Resistors_THT:R_Axial_DIN0207_L6.3mm_D2.5mm_P7.62mm_Horizontal
- resetButton_1: footprint (none) -> Pin_Headers:Pin_Header_Angled_1x02_Pitch2.54mm
- gave numbers to parts that had none: 2
Connections:
- net ALIM_TOF: now also JP203.1, JP204.1; no longer J_TOF201.2 (P2), J_TOF202.2 (P2)
- net GND: now also J203.3 (Pin_3), J204.2 (Pin_2), J205.1 (Pin_1), J205.4 (Pin_4)
- net at JP204.2: now also J_TOF202.2 (P2)
- net at JP203.2: now also J_TOF201.2 (P2)
- new net 3.3V_ext: J205.3 (Pin_3)
- new net 5V_ext: J205.2 (Pin_2)
- new net ALIM_UC: J203.2 (Pin_2)
- new net GPIO_EXT5: J204.1 (Pin_1)
- new net ICSPCLK: J203.5 (Pin_5)
- new net ICSPDAT: J203.4 (Pin_4)
- new net P_RESET: J203.1 (Pin_1)
- no-connect marks 31 -> 32
Other:
- moved on the sheet: JP203, JP204, J_EXT201, J_EXT202, J_SERV201, J_TOF202
