File: shieldNumero9.kicad_pcb (KiCad board)
At the start: 2 copper layers, 98 x 82 mm, 19 parts, among them J201 Conn_01x06, J202 Conn_01x06, U401 7805, U402 LF33CDT-TRY

Commit message: finish schematics. add componants, find right chip, firest verification OK, ready for routing
Parts:
- added C401: C, Capacitors_THT:C_Disc_D3.8mm_W2.6mm_P2.50mm, F.Cu at (200.9, 27.4)
- added C402: C, Capacitors_THT:C_Disc_D3.8mm_W2.6mm_P2.50mm, F.Cu at (194.8, 39.1)
- added C403: C, Capacitors_THT:C_Disc_D3.8mm_W2.6mm_P2.50mm, F.Cu at (201.2, 40.1)
- added C404: C, Capacitors_THT:C_Disc_D3.8mm_W2.6mm_P2.50mm, F.Cu at (205.2, 32.8)
- added J203: Conn_01x06, Pin_Headers:Pin_Header_Straight_1x06_Pitch2.54mm, F.Cu at (178.8, 96.8)
- added J204: Conn_01x02, Pin_Headers:Pin_Header_Straight_1x02_Pitch2.54mm, F.Cu at (246.9, 47.0)
- added J205: Conn_01x04, Socket_Strips:Socket_Strip_Straight_1x04_Pitch2.54mm, F.Cu at (262.6, 36.3)
- added JP203: Jumper, Pin_Headers:Pin_Header_Straight_2x01_Pitch2.54mm, F.Cu at (88.4, 109.7)
- added JP204: Jumper, Pin_Headers:Pin_Header_Straight_2x01_Pitch2.54mm, F.Cu at (54.4, 109.5)
- added LED501: LED, LEDs:LED_D5.0mm, F.Cu at (184.9, 129.0)
- added LED502: LED, LEDs:LED_D5.0mm, F.Cu at (184.9, 137.9)
- added LED503: LED, LEDs:LED_D5.0mm, F.Cu at (185.9, 147.1)
- added R501: R, Resistors_THT:R_Axial_DIN0207_L6.3mm_D2.5mm_P7.62mm_Horizontal, F.Cu at (219.5, 112.3)
- added R502: R, Resistors_THT:R_Axial_DIN0207_L6.3mm_D2.5mm_P7.62mm_Horizontal, F.Cu at (201.7, 117.9)
- added R503: R, Resistors_THT:R_Axial_DIN0207_L6.3mm_D2.5mm_P7.62mm_Horizontal, F.Cu at (204.0, 92.2)
- added R504: R, Resistors_THT:R_Axial_DIN0207_L6.3mm_D2.5mm_P7.62mm_Horizontal, F.Cu at (192.5, 130.3)
- added R505: R, Resistors_THT:R_Axial_DIN0207_L6.3mm_D2.5mm_P7.62mm_Horizontal, F.Cu at (192.0, 138.9)
- added R506: R, Resistors_THT:R_Axial_DIN0207_L6.3mm_D2.5mm_P7.62mm_Horizontal, F.Cu at (193.0, 146.6)
- added R_pullup_reset_esp_1: R, Resistors_THT:R_Axial_DIN0207_L6.3mm_D2.5mm_P7.62mm_Horizontal, F.Cu at (74.2, -17.0)
- added SW501: SW_Push, Buttons_Switches_THT:SW_PUSH_6mm, F.Cu at (218.4, 100.8)
- added SW502: SW_Push, Buttons_Switches_THT:SW_PUSH_6mm, F.Cu at (205.7, 107.7)
- added SW503: SW_Push, Buttons_Switches_THT:SW_PUSH_6mm, F.Cu at (204.7, 97.5)
- added U301: Pic16f15345, Housings_DIP:DIP-20_W7.62mm_LongPads, F.Cu at (186.9, 93.2)
- added resetButton_1: Conn_01x02, Pin_Headers:Pin_Header_Angled_1x02_Pitch2.54mm, F.Cu at (87.4, -13.7)
- moved J_SERV201 99.1 mm to (248.7, 81.3)
- moved U401 54.3 mm to (191.8, 32.5)
- moved U402 54.3 mm to (191.9, 21.8)
- moved JP201 0.35 mm to (4.06, 88.4)
Connections:
- net ALIM_UC renamed 3.3V_ext
- J_TOF201 pad 2: 5V_SERVO -> Net-(JP203-Pad2)
- J_TOF202 pad 2: 5V_SERVO -> Net-(JP204-Pad2)
- J_arduino0-7_202 pad 6: Net-(J_arduino0-7_202-Pad6) -> Arduino-CTRLTOFXSHUT
Other:
- outline, holes or cut-outs redrawn
- board text added: "TODO : - ajouter des fixations mecaniques pour extention / protection - ajouter du texte sur la board - ajouter un trou pour le servo"

Commit message: placement componants seems OK
Parts:
- moved J_EXT202 229.4 mm to (27.9, 25.4)
- moved J204 224.5 mm to (27.9, 96.5)
- moved J_SERV201 183.1 mm to (68.6, 48.3)
- moved R501 174.0 mm to (48.3, 81.3)
- moved SW501 159.4 mm to (61.0, 76.2)
- moved R502 159.0 mm to (48.3, 76.2)
- moved R503 156.3 mm to (48.3, 78.7)
- moved J205 155.9 mm to (116.8, 91.4)
- moved R506 154.0 mm to (68.6, 55.9)
- moved R505 147.4 mm to (68.6, 58.4)
- moved R504 142.0 mm to (68.6, 61.0)
- moved LED503 139.1 mm to (71.1, 68.6)
- moved SW503 135.3 mm to (71.1, 76.2)
- moved J203 133.1 mm to (48.3, 71.1), turned to 180 degrees
- moved J_EXT201 130.5 mm to (116.8, 25.4)
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Other:
- board text added: "3.3 V ESP GND"
- board text added: "5V \/ 3.3 /\"
- board text added: "ESP 8266"
- board text added: "Enable TOF2 Enable TOF1"
- board text added: "GPIO0 GPIO2 Reset CH_PD"
- board text added: "JY-MCU"
- board text added: "TOF1"
- board text added: "TOF2"
- board text added: "TX arduino RX Arduino"

Commit message: finish routing, need to double check
Parts:
- moved C403 5.74 mm to (88.8, 88.9), turned to 90 degrees
Routing:
- net GND: track 0.00 -> 572.5 mm
- net Arduino-SDA: track 0.00 -> 193.3 mm
- net 3.3V_ext: track 0.00 -> 188.4 mm
- net Shield-ALIM+: track 0.00 -> 168.5 mm, vias 0 -> 1
- net 5V_SERVO: track 0.00 -> 164.8 mm
- net Arduino-SCL: track 0.00 -> 135.1 mm
- net TX_arduino_5V: track 0.00 -> 126.8 mm
- net RX_ardunio_5V: track 0.00 -> 125.4 mm
- net Arduino-CTRLTOFXSHUT: track 0.00 -> 123.8 mm
- net GPIO_EXT5: track 0.00 -> 105.4 mm
- net P_BUT2: track 0.00 -> 63.8 mm
- net 3.3-CTRLTOFXSHUT: track 0.00 -> 59.7 mm, vias 0 -> 1
- net P_RESET: track 0.00 -> 52.5 mm, vias 0 -> 1
- net /IO shield/ESP-RESET: track 0.00 -> 47.7 mm
- net GPIO_EXT1: track 0.00 -> 44.5 mm
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- added copper zone on F.Cu, net GND

Commit message: add file for fab
Parts:
- added REF**: 1pin, Connectors:1pin, F.Cu at (112.0, 31.0)
- added REF**: 1pin, Connectors:1pin, F.Cu at (112.0, 93.0)
- added REF**: 1pin, Connectors:1pin, F.Cu at (34.0, 93.0)
- added REF**: 1pin, Connectors:1pin, F.Cu at (40.0, 31.0)
- moved C403 2.67 mm to (91.4, 88.9)
Routing:
- net 3.3V_ext: track 188.4 -> 281.3 mm
- net 3.3-CTRLTOFXSHUT: track 59.7 -> 96.6 mm, vias 1 -> 0
- net Net-(JP203-Pad2): track 25.6 -> 47.8 mm
- net 5V_SERVO: track 164.8 -> 174.4 mm
- net Shield-ALIM+: track 168.5 -> 176.9 mm
- net GPIO_EXT1: track 44.5 -> 49.7 mm
- net GPIO_EXT2: track 44.3 -> 41.1 mm
- net GPIO_EXT3: track 44.0 -> 41.5 mm
- net Arduino-CTRLTOFXSHUT: track 123.8 -> 125.6 mm
- net RX_ardunio_5V: track 125.4 -> 127.2 mm
- net TX_arduino_5V: track 126.8 -> 128.5 mm
- net GPIO_EXT4: track 43.0 -> 41.5 mm
- net GPIO_EXT5: track 105.4 -> 104.3 mm
- net Net-(JP204-Pad2): track 26.1 -> 26.7 mm
Other:
- board text added: "#9"
- board text added: "Numero 9 carte extension V1 11-03-2018"
- board text removed: "TODO : - ajouter des fixations mecaniques pour extention / protection - ajouter du texte sur la board - ajouter un trou pour le servo"
